File: pcb/pulse_gen.kicad_pcb (KiCad board)
At the start: 4 copper layers, 45 x 45 mm, 27 parts, among them J1 Screw_Terminal_01x02, J2 USB_B, J3 Conn_Coaxial, U1 74AC14, U2 LD1117S33TR_SOT223

Commit message: Update to KiCAD v9 etc.
Parts:
- removed LOGO1: LOGO_SH_SMALL, 01_Sebastian:SebastianHarnisch_small
Other:
- board text added: "SEBASTIAN HARNISCH"
