File: pcb/pulse_gen.kicad_sch (KiCad schematic)
At the start: 27 parts, among them J1 Screw_Terminal_01x02, J2 USB_B, J3 Conn_Coaxial, U1 74AC14, U2 LD1117S33TR_SOT223

Commit message: Update to KiCAD v9 etc.
Parts:
- removed LOGO1: LOGO_SH_SMALL, 01_Sebastian:SebastianHarnisch_small, symbol 01_Sebastian:LOGO_SH_SMALL
Changed lines of the file:
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@@
 (kicad_sch
-	(version 20231120)
+	(version 20250114)
 	(generator "eeschema")
-	(generator_version "8.0")
+	(generator_version "9.0")
 	(paper "A4")
 	(title_block
@@
 		(comment 1 "Pulse gen circuit presented by W2AEW")
 	)
+	(text "Power supply"
+		(exclude_from_sim no)
+		(at 21.59 21.59 0)
+		(effects
+			(font
+				(size 1.27 1.27)
+			)
+			(justify left bottom)
+		)
+	)
+	(text "Inverter oscillator/buffer"
+		(exclude_from_sim no)
+		(at 21.59 95.25 0)
+		(effects
+			(font
+				(size 1.27 1.27)
+			)
+			(justify left bottom)
+		)
+	)
 	(junction
 		(at 64.77 132.08)
@@
 		)
 	)
-	(text "Power supply"
-		(exclude_from_sim no)
-		(at 21.59 21.59 0)
-		(effects
-			(font
-				(size 1.27 1.27)
-			)
-			(justify left bottom)
-		)
-	)
-	(text "Inverter oscillator/buffer"
-		(exclude_from_sim no)
-		(at 21.59 95.25 0)
-		(effects
-			(font
-				(size 1.27 1.27)
-			)
-			(justify left bottom)
-		)
-	)
 	(symbol
 		(lib_id "74xx:74HC14")
@@
 	)
 	(symbol
-		(lib_id "01_Sebastian:LOGO_SH_SMALL")
-		(at 210.82 156.21 0)
-		(unit 1)
-		(exclude_from_sim no)
-		(in_bom yes)
-		(on_board yes)
-		(dnp no)
-		(fields_autoplaced yes)
-		(property "Reference" "LOGO1"
-			(at 210.82 152.4 0)
-			(effects
-				(font
-					(size 1.27 1.27)
-				)
-				(hide yes)
-			)
-		)
-		(property "Value" "LOGO_SH_SMALL"
-			(at 212.09 160.02 0)
-			(effects
-				(font
-					(size 1.27 1.27)
-				)
-				(hide yes)
-			)
-		)
-		(property "Footprint" "01_Sebastian:SebastianHarnisch_small"
-			(at 210.82 162.56 0)
-			(effects
-				(font
-					(size 1.27 1.27)
-				)
-				(hide yes)
-			)
-		)
-		(property "Datasheet" ""
-			(at 210.82 157.48 0)
-			(effects
-				(font
-					(size 1.27 1.27)
-				)
-				(hide yes)
-			)
-		)
-		(property "Description" ""
-			(at 210.82 156.21 0)
-			(effects
-				(font
-					(size 1.27 1.27)
-				)
-				(hide yes)
-			)
-		)
-		(instances
-			(project "pulse_gen"
-				(path "/17b43078-d0d1-4ab8-81ac-be1bc5ec3fd8"
-					(reference "LOGO1")
-					(unit 1)
-				)
-			)
-		)
-	)
-	(symbol
 		(lib_id "power:GND")
 		(at 187.96 140.97 0)
@@
 		)
 	)
+	(embedded_fonts no)
 )
